File: kicad/LDO.kicad_sch (KiCad schematic)
At the start: 6 parts, among them U2 RT9069-33GB

Commit message: Some random tildas added by default for some reason
Parts:
- D1: value (none) -> ~
Changed lines of the file:
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@@
       (effects (font (size 1.27 1.27)) (justify left))
     )
-    (property "Value" "" (id 1) (at 149.86 102.87 0)
+    (property "Value" "~" (id 1) (at 149.86 102.87 0)
       (effects (font (size 1.524 1.524)) hide)
     )

Commit message: Some overwritten changes by swapping back to robot project
Parts:
- D1: value ~ -> LTST-C190KGKT; footprint (none) -> digikey-footprints:LED_0603
Changed lines of the file:
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@@
       (effects (font (size 1.27 1.27)) (justify left))
     )
-    (property "Value" "~" (id 1) (at 149.86 102.87 0)
+    (property "Value" "LTST-C190KGKT" (id 1) (at 149.86 102.87 0)
       (effects (font (size 1.524 1.524)) hide)
     )
-    (property "Footprint" "" (id 2) (at 158.75 107.95 0)
+    (property "Footprint" "digikey-footprints:LED_0603" (id 2) (at 158.75 107.95 0)
       (effects (font (size 1.524 1.524)) (justify left) hide)
     )

Commit message: removed value from diode
Parts:
- D1: value LTST-C190KGKT -> ~
Changed lines of the file:
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@@
       (effects (font (size 1.27 1.27)) (justify left))
     )
-    (property "Value" "LTST-C190KGKT" (id 1) (at 149.86 102.87 0)
+    (property "Value" "~" (id 1) (at 149.86 102.87 0)
       (effects (font (size 1.524 1.524)) hide)
     )

Commit message: wip prior to moving back to work on docs
Parts:
- D1: value ~ -> LTST-C190KGKT
Changed lines of the file:
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@@
       (effects (font (size 1.27 1.27)) (justify left))
     )
-    (property "Value" "~" (id 1) (at 149.86 102.87 0)
+    (property "Value" "LTST-C190KGKT" (id 1) (at 149.86 102.87 0)
       (effects (font (size 1.524 1.524)) hide)
     )
