File: kicad/Top/HostInterface.kicad_sch (KiCad schematic)
At the start: 8 parts

Commit message: Properly synced pcb to schematic
Parts:
- J8: value ~ -> 0022053041; footprint CONN_22-05-3041 -> AltiumImports:CONN_22-05-3041
- J9: value ~ -> N2510-6002-RB; footprint CONN_2510-6002 -> AltiumImports:CONN_2510-6002
- JP33, JP36: value ~ -> Header_2x1; footprint CONN_PEC02SAAN -> AltiumImports:CONN_PEC02SAAN
- R39, R46: value ~ -> ERJ-8ENF10R0V; footprint 1206 -> AltiumImports:1206
- R42, R43: value ~ -> CRCW040210K0FKED; footprint 0402 -> AltiumImports:0402
Changed lines of the file:
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@@
   (symbol (lib_id "Top-altium-import:AGND") (at 96.52 132.08 0) (unit 1)
     (in_bom yes) (on_board yes)
-    (property "Reference" "#PWR?" (id 0) (at 96.52 132.08 0)
+    (property "Reference" "#PWR0265" (id 0) (at 96.52 132.08 0)
       (effects (font (size 1.27 1.27)) hide)
     )
@@
   (symbol (lib_id "Top-altium-import:3V3_U2") (at 114.3 86.36 180) (unit 1)
     (in_bom yes) (on_board yes)
-    (property "Reference" "#PWR?" (id 0) (at 114.3 86.36 0)
+    (property "Reference" "#PWR0261" (id 0) (at 114.3 86.36 0)
       (effects (font (size 1.27 1.27)) hide)
     )
@@
   (symbol (lib_id "Top-altium-import:AGND") (at 152.4 137.16 0) (unit 1)
     (in_bom yes) (on_board yes)
-    (property "Reference" "#PWR?" (id 0) (at 152.4 137.16 0)
+    (property "Reference" "#PWR0264" (id 0) (at 152.4 137.16 0)
       (effects (font (size 1.27 1.27)) hide)
     )
@@
       (effects (font (size 1.27 1.27)) (justify left bottom))
     )
-    (property "Value" "~" (id 1) (at 137.16 139.7 0)
-      (effects (font (size 1.27 1.27)) (justify left bottom) hide)
-    )
-    (property "Footprint" "CONN_22-05-3041" (id 2) (at 142.24 132.08 0)
+    (property "Value" "0022053041" (id 1) (at 137.16 139.7 0)
+      (effects (font (size 1.27 1.27)) (justify left bottom) hide)
+    )
+    (property "Footprint" "AltiumImports:CONN_22-05-3041" (id 2) (at 142.24 132.08 0)
       (effects (font (size 1.27 1.27)) hide)
     )
@@
       (effects (font (size 1.27 1.27)) (justify left bottom))
     )
-    (property "Value" "~" (id 1) (at 103.378 93.472 0)
-      (effects (font (size 1.27 1.27)) (justify left bottom) hide)
-    )
-    (property "Footprint" "0402" (id 2) (at 104.14 99.06 0)
+    (property "Value" "CRCW040210K0FKED" (id 1) (at 103.378 93.472 0)
+      (effects (font (size 1.27 1.27)) (justify left bottom) hide)
+    )
+    (property "Footprint" "AltiumImports:0402" (id 2) (at 104.14 99.06 0)
       (effects (font (size 1.27 1.27)) hide)
     )
@@
   (symbol (lib_id "Top-altium-import:AGND") (at 90.17 58.42 0) (unit 1)
     (in_bom yes) (on_board yes)
-    (property "Reference" "#PWR?" (id 0) (at 90.17 58.42 0)
+    (property "Reference" "#PWR0266" (id 0) (at 90.17 58.42 0)
       (effects (font (size 1.27 1.27)) hide)
     )
@@
   (symbol (lib_id "Top-altium-import:3V3_U2") (at 35.56 132.08 270) (unit 1)
     (in_bom yes) (on_board yes)
-    (property "Reference" "#PWR?" (id 0) (at 35.56 132.08 0)
+    (property "Reference" "#PWR0267" (id 0) (at 35.56 132.08 0)
       (effects (font (size 1.27 1.27)) hide)
     )
@@
       (effects (font (size 1.27 1.27)) (justify left bottom))
     )
-    (property "Value" "~" (id 1) (at 156.21 128.27 0)
-      (effects (font (size 1.27 1.27)) (justify left bottom) hide)
-    )
-    (property "Footprint" "1206" (id 2) (at 157.48 124.46 0)
+    (property "Value" "ERJ-8ENF10R0V" (id 1) (at 156.21 128.27 0)
+      (effects (font (size 1.27 1.27)) (justify left bottom) hide)
+    )
+    (property "Footprint" "AltiumImports:1206" (id 2) (at 157.48 124.46 0)
       (effects (font (size 1.27 1.27)) hide)
     )
@@
   (symbol (lib_id "Top-altium-import:3V3_U2") (at 149.86 66.04 90) (unit 1)
     (in_bom yes) (on_board yes)
-    (property "Reference" "#PWR?" (id 0) (at 149.86 66.04 0)
+    (property "Reference" "#PWR0262" (id 0) (at 149.86 66.04 0)
       (effects (font (size 1.27 1.27)) hide)
     )
@@
       (effects (font (size 1.27 1.27)) (justify left bottom))
     )
-    (property "Value" "~" (id 1) (at 43.18 121.92 0)
-      (effects (font (size 1.27 1.27)) (justify left bottom) hide)
-    )
-    (property "Footprint" "CONN_PEC02SAAN" (id 2) (at 48.26 127 0)
+    (property "Value" "Header_2x1" (id 1) (at 43.18 121.92 0)
+      (effects (font (size 1.27 1.27)) (justify left bottom) hide)
+    )
+    (property "Footprint" "AltiumImports:CONN_PEC02SAAN" (id 2) (at 48.26 127 0)
       (effects (font (size 1.27 1.27)) hide)
     )
@@
       (effects (font (size 1.27 1.27)) (justify left bottom))
     )
-    (property "Value" "~" (id 1) (at 68.072 124.46 0)
-      (effects (font (size 1.27 1.27)) (justify left bottom) hide)
-    )
-    (property "Footprint" "CONN_2510-6002" (id 2) (at 78.74 132.08 0)
+    (property "Value" "N2510-6002-RB" (id 1) (at 68.072 124.46 0)
+      (effects (font (size 1.27 1.27)) (justify left bottom) hide)
+    )
+    (property "Footprint" "AltiumImports:CONN_2510-6002" (id 2) (at 78.74 132.08 0)
       (effects (font (size 1.27 1.27)) hide)
     )
@@
   (symbol (lib_id "Top-altium-import:3V3_U2") (at 177.8 124.46 90) (unit 1)
     (in_bom yes) (on_board yes)
-    (property "Reference" "#PWR?" (id 0) (at 177.8 124.46 0)
+    (property "Reference" "#PWR0263" (id 0) (at 177.8 124.46 0)
       (effects (font (size 1.27 1.27)) hide)
     )
@@
       (effects (font (size 1.27 1.27)) (justify left bottom))
     )
-    (property "Value" "~" (id 1) (at 123.698 93.472 0)
-      (effects (font (size 1.27 1.27)) (justify left bottom) hide)
-    )
-    (property "Footprint" "0402" (id 2) (at 124.46 99.06 0)
+    (property "Value" "CRCW040210K0FKED" (id 1) (at 123.698 93.472 0)
+      (effects (font (size 1.27 1.27)) (justify left bottom) hide)
+    )
+    (property "Footprint" "AltiumImports:0402" (id 2) (at 124.46 99.06 0)
       (effects (font (size 1.27 1.27)) hide)
     )
@@
       (effects (font (size 1.27 1.27)) (justify left bottom))
     )
-    (property "Value" "~" (id 1) (at 52.832 131.318 0)
-      (effects (font (size 1.27 1.27)) (justify left bottom) hide)
-    )
-    (property "Footprint" "1206" (id 2) (at 58.42 132.08 0)
+    (property "Value" "ERJ-8ENF10R0V" (id 1) (at 52.832 131.318 0)
+      (effects (font (size 1.27 1.27)) (justify left bottom) hide)
+    )
+    (property "Footprint" "AltiumImports:1206" (id 2) (at 58.42 132.08 0)
       (effects (font (size 1.27 1.27)) hide)
     )
@@
       (effects (font (size 1.27 1.27)) (justify left bottom))
     )
-    (property "Value" "~" (id 1) (at 167.64 114.3 0)
-      (effects (font (size 1.27 1.27)) (justify left bottom) hide)
-    )
-    (property "Footprint" "CONN_PEC02SAAN" (id 2) (at 170.18 119.38 0)
-      (effects (font (size 1.27 1.27)) hide)
-    )
+    (property "Value" "Header_2x1" (id 1) (at 167.64 114.3 0)
+      (effects (font (size 1.27 1.27)) (justify left bottom) hide)
+    )
+    (property "Footprint" "AltiumImports:CONN_PEC02SAAN" (id 2) (at 170.18 119.38 0)
+      (effects (font (size 1.27 1.27)) hide)
+    )
