File: kicad/Top/Hardware.kicad_sch (KiCad schematic)
At the start: 39 parts

Commit message: Properly synced pcb to schematic
Parts:
- FID1, FID2, FID3, FID4, FID5, FID6: value ~ -> CMP-0077181-1; footprint Fiducial10-20 -> AltiumImports:Fiducial10-20
- H1, H2, H3, H4: value ~ -> SJ-5303 (CLEAR); footprint Bumpon_SJ5003Transparent -> AltiumImports:Bumpon_SJ5003Transparent
- LOGO5: value ~ -> CAUTION HOT SURFACE; footprint IEC_HotSurface_Small -> AltiumImports:IEC_HotSurface_Small
- SH-JP1: value ~ -> ACDRV1 to _acdrv1; footprint FP-SNT-100-BK-G-MFG -> AltiumImports:FP-SNT-100-BK-G-MFG
- SH-JP10, SH-JP11, SH-JP12, SH-JP14, SH-JP16, SH-JP19, SH-JP32, SH-JP34, SH-JP35, SH-JP36, SH-JP37, SH-JP6, SH-JP9: value ~ -> Installed; footprint FP-SNT-100-BK-G-MFG -> AltiumImports:FP-SNT-100-BK-G-MFG
- SH-JP13, SH-JP15, SH-JP23, SH-JP24, SH-JP25, SH-JP3, SH-JP33, SH-JP4, SH-JP5: value ~ -> Not Installed; footprint FP-SNT-100-BK-G-MFG -> AltiumImports:FP-SNT-100-BK-G-MFG
- SH-JP2: value ~ -> ACDRV2 to _acdrv2; footprint FP-SNT-100-BK-G-MFG -> AltiumImports:FP-SNT-100-BK-G-MFG
- ZZ1: value ~ -> These assemblies are ESD sensitive, ESD precautions shall be observed.; footprint AssemblyNote -> AltiumImports:AssemblyNote
- ZZ2: value ~ -> These assemblies must be clean and free from flux and all contaminants. Use of no clean flux is not acceptable.; footprint AssemblyNote -> AltiumImports:AssemblyNote
- ZZ3: value ~ -> These assemblies must comply with workmanship standards IPC-A-610 Class 2, unless otherwise specified.; footprint AssemblyNote -> AltiumImports:AssemblyNote
