File: kicad/robot/usb-c-phonepc.kicad_sch (KiCad schematic)
At the start: 11 parts, among them J4 USB4120-03-C_REVA

Commit message: WARNING Major BOM cleanup
Parts:
- J4: MANUFACTURER GCT -> (none); Manufacturer (none) -> GCT
- TP13: value D- -> TP5002
- TP14: value D+ -> TP5002
- TP15: value CC1 -> TP5002
- TP29: value CC2 -> TP5002
- TP30: value VBUS -> TP5002
Changed lines of the file:
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@@
       (effects (font (size 1.27 1.27)) (justify left bottom) hide)
     )
-    (property "MANUFACTURER" "GCT" (id 7) (at 91.44 96.52 0)
+    (property "MANUFACTURER" "" (id 7) (at 91.44 96.52 0)
       (effects (font (size 1.27 1.27)) (justify left bottom) hide)
     )
     (property "Part Number" "USB4120-03-C" (id 8) (at 91.44 96.52 0)
+      (effects (font (size 1.27 1.27)) hide)
+    )
+    (property "Manufacturer" "GCT" (id 9) (at 91.44 96.52 0)
       (effects (font (size 1.27 1.27)) hide)
     )
@@
       (effects (font (size 1.27 1.27)) (justify left))
     )
-    (property "Value" "VBUS" (id 1) (at 222.25 68.58 0)
+    (property "Value" "TP5002" (id 1) (at 222.25 68.58 0)
       (effects (font (size 1.27 1.27)) (justify left))
     )
@@
     )
     (property "Datasheet" "~" (id 3) (at 224.79 71.12 0)
+      (effects (font (size 1.27 1.27)) hide)
+    )
+    (property "Description" "PPC_VBUS" (id 4) (at 219.71 71.12 0)
       (effects (font (size 1.27 1.27)) hide)
     )
@@
       (effects (font (size 1.27 1.27)) (justify left))
     )
-    (property "Value" "CC1" (id 1) (at 144.78 77.47 0)
+    (property "Value" "TP5002" (id 1) (at 144.78 77.47 0)
       (effects (font (size 1.27 1.27)) (justify left))
     )
@@
       (effects (font (size 1.27 1.27)) (justify left))
     )
-    (property "Value" "D+" (id 1) (at 109.22 110.49 0)
+    (property "Value" "TP5002" (id 1) (at 109.22 110.49 0)
       (effects (font (size 1.27 1.27)) (justify left))
     )
@@
     )
     (property "Datasheet" "~" (id 3) (at 111.76 113.03 0)
+      (effects (font (size 1.27 1.27)) hide)
+    )
+    (property "Description" "PPC_D+" (id 4) (at 106.68 113.03 0)
       (effects (font (size 1.27 1.27)) hide)
     )
@@
       (effects (font (size 1.27 1.27)) (justify left))
     )
-    (property "Value" "D-" (id 1) (at 109.22 99.5679 0)
+    (property "Value" "TP5002" (id 1) (at 109.22 99.5679 0)
       (effects (font (size 1.27 1.27)) (justify left))
     )
@@
       (effects (font (size 1.27 1.27)) hide)
     )
+    (property "Description" "PPC_D-" (id 4) (at 106.68 101.6 0)
+      (effects (font (size 1.27 1.27)) hide)
+    )
     (pin "1")
   )
@@
       (effects (font (size 1.27 1.27)) (justify right))
     )
-    (property "Value" "CC2" (id 1) (at 144.78 87.63 0)
+    (property "Value" "TP5002" (id 1) (at 144.78 87.63 0)
       (effects (font (size 1.27 1.27)) (justify right))
     )
@@
       (effects (font (size 1.27 1.27)) hide)
     )
+    (property "Description" "CC2" (id 4) (at 142.24 82.55 0)
+      (effects (font (size 1.27 1.27)) hide)
+    )

Commit message: WARNING more BOM batch edits
Parts:
- TP13, TP14, TP15, TP29, TP30: Manufacturer (none) -> Keystone Electronics; Part Number (none) -> 5002
Changed lines of the file:
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@@
+      (effects (font (size 1.27 1.27)) hide)
+    )
+    (property "Manufacturer" "Keystone Electronics" (id 5) (at 219.71 71.12 0)
+      (effects (font (size 1.27 1.27)) hide)
+    )
+    (property "Part Number" "5002" (id 6) (at 219.71 71.12 0)
       (effects (font (size 1.27 1.27)) hide)
     )
@@
     )
     (property "Datasheet" "~" (id 3) (at 147.32 80.01 0)
+      (effects (font (size 1.27 1.27)) hide)
+    )
+    (property "Manufacturer" "Keystone Electronics" (id 4) (at 142.24 80.01 0)
+      (effects (font (size 1.27 1.27)) hide)
+    )
+    (property "Part Number" "5002" (id 5) (at 142.24 80.01 0)
       (effects (font (size 1.27 1.27)) hide)
     )
@@
       (effects (font (size 1.27 1.27)) hide)
     )
+    (property "Manufacturer" "Keystone Electronics" (id 5) (at 106.68 113.03 0)
+      (effects (font (size 1.27 1.27)) hide)
+    )
+    (property "Part Number" "5002" (id 6) (at 106.68 113.03 0)
+      (effects (font (size 1.27 1.27)) hide)
+    )
     (pin "1")
   )
@@
     )
     (property "Description" "PPC_D-" (id 4) (at 106.68 101.6 0)
+      (effects (font (size 1.27 1.27)) hide)
+    )
+    (property "Manufacturer" "Keystone Electronics" (id 5) (at 106.68 101.6 0)
+      (effects (font (size 1.27 1.27)) hide)
+    )
+    (property "Part Number" "5002" (id 6) (at 106.68 101.6 0)
       (effects (font (size 1.27 1.27)) hide)
     )
@@
       (effects (font (size 1.27 1.27)) hide)
     )
+    (property "Manufacturer" "Keystone Electronics" (id 5) (at 142.24 82.55 0)
+      (effects (font (size 1.27 1.27)) hide)
+    )
+    (property "Part Number" "5002" (id 6) (at 142.24 82.55 0)
+      (effects (font (size 1.27 1.27)) hide)
+    )

Commit message: Batch BOM edits adding manufactuer and part numbers only
Parts:
- D3: Manufacturer (none) -> Nexperia
Changed lines of the file:
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@@
+      (effects (font (size 1.27 1.27)) hide)
+    )
+    (property "Manufacturer" "Nexperia" (id 6) (at 194.31 81.28 0)
       (effects (font (size 1.27 1.27)) hide)
     )

Commit message: bulk BOM edits. Mainly dealing with cap voltage ratings and part selection
Parts:
- C89, C95: Manufacturer (none) -> Murata; Part Number (none) -> GRM1555C1H270JA01J
- C97: Manufacturer (none) -> Samsung; Part Number (none) -> CL21B225KBYNNNE
Changed lines of the file:
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@@
     )
     (property "Description" "35V" (id 4) (at 217.17 82.55 0))
+    (property "Manufacturer" "Samsung" (id 5) (at 212.09 78.74 0)
+      (effects (font (size 1.27 1.27)) hide)
+    )
+    (property "Part Number" "CL21B225KBYNNNE" (id 6) (at 212.09 78.74 0)
+      (effects (font (size 1.27 1.27)) hide)
+    )
     (pin "1")
     (pin "2")
@@
       (effects (font (size 1.27 1.27)) hide)
     )
+    (property "Manufacturer" "Murata" (id 5) (at 137.16 92.71 0)
+      (effects (font (size 1.27 1.27)) hide)
+    )
+    (property "Part Number" "GRM1555C1H270JA01J" (id 6) (at 137.16 92.71 0)
+      (effects (font (size 1.27 1.27)) hide)
+    )
     (pin "1")
     (pin "2")
@@
       (effects (font (size 1.27 1.27)) hide)
     )
+    (property "Manufacturer" "Murata" (id 5) (at 124.46 92.71 0)
+      (effects (font (size 1.27 1.27)) hide)
+    )
+    (property "Part Number" "GRM1555C1H270JA01J" (id 6) (at 124.46 92.71 0)
+      (effects (font (size 1.27 1.27)) hide)
+    )
