File: kicad/robot/Protection.kicad_sch (KiCad schematic)
At the start: 23 parts, among them Q2 EFC8811R-TF, U12 BQ27742YZFR-G1

Commit message: WARNING Major BOM cleanup
Parts:
- BT1: Part Number 103AT-5-1P-FT -> 103AT-5-1P-FT
Changed lines of the file:
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@@
       (effects (font (size 1.27 1.27)) hide)
     )
-    (property "Part Number" " 103AT-5-1P-FT " (id 4) (at 106.68 163.83 0)
+    (property "Part Number" "103AT-5-1P-FT" (id 4) (at 106.68 163.83 0)
       (effects (font (size 1.27 1.27)) hide)
     )
@@
       (effects (font (size 1.27 1.27)) hide)
     )
-    (property "Part Number" " 103AT-5-1P-FT " (id 4) (at 106.68 163.83 0)
+    (property "Part Number" "103AT-5-1P-FT" (id 4) (at 106.68 163.83 0)
       (effects (font (size 1.27 1.27)) hide)
     )

Commit message: WARNING more BOM batch edits
Parts:
- Q2: Part Number (none) -> EFC8811R-TF
- R43, R45: Manufacturer (none) -> Bourns; Part Number (none) -> CR0402-JW-201GLF
- R48: Manufacturer (none) -> Stackpole Electronics; Part Number (none) -> RMCF0603FT2K00
- U12: Part Number (none) -> BQ27742YZFR-G1
Changed lines of the file:
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@@
       (effects (font (size 1.27 1.27)) (justify left) hide)
+    )
+    (property "Part Number" "EFC8811R-TF" (id 34) (at 264.16 105.41 0)
+      (effects (font (size 1.27 1.27)) hide)
     )
     (pin "1")
@@
     (property "temperature range low" "-40°C" (id 34) (at 158.75 35.56 0)
       (effects (font (size 1.27 1.27)) (justify left) hide)
+    )
+    (property "Part Number" "BQ27742YZFR-G1" (id 35) (at 158.75 127 0)
+      (effects (font (size 1.27 1.27)) hide)
     )
     (pin "A1")
@@
       (effects (font (size 1.27 1.27)) hide)
     )
+    (property "Manufacturer" "Bourns" (id 4) (at 218.44 90.17 0)
+      (effects (font (size 1.27 1.27)) hide)
+    )
+    (property "Part Number" "CR0402-JW-201GLF" (id 5) (at 218.44 90.17 0)
+      (effects (font (size 1.27 1.27)) hide)
+    )
     (pin "1")
     (pin "2")
@@
       (effects (font (size 1.27 1.27)) hide)
     )
+    (property "Manufacturer" "Stackpole Electronics" (id 4) (at 287.02 114.3 0)
+      (effects (font (size 1.27 1.27)) hide)
+    )
+    (property "Part Number" "RMCF0603FT2K00" (id 5) (at 287.02 114.3 0)
+      (effects (font (size 1.27 1.27)) hide)
+    )
     (pin "1")
     (pin "2")
@@
       (effects (font (size 1.27 1.27)) hide)
     )
+    (property "Manufacturer" "Bourns" (id 4) (at 238.76 90.17 0)
+      (effects (font (size 1.27 1.27)) hide)
+    )
+    (property "Part Number" "CR0402-JW-201GLF" (id 5) (at 238.76 90.17 0)
+      (effects (font (size 1.27 1.27)) hide)
+    )

Commit message: Added stock counts to parts I have
Parts:
- Q2, U12: Stock (none) -> 25
Changed lines of the file:
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@@
+      (effects (font (size 1.27 1.27)) hide)
+    )
+    (property "Stock" "25" (id 35) (at 264.16 105.41 0)
       (effects (font (size 1.27 1.27)) hide)
     )
@@
       (effects (font (size 1.27 1.27)) hide)
     )
+    (property "Stock" "25" (id 36) (at 158.75 127 0)
+      (effects (font (size 1.27 1.27)) hide)
+    )

Commit message: Batch BOM edits adding manufactuer and part numbers only
Parts:
- BT1: Manufacturer (none) -> Semitec
- Q2: Manufacturer (none) -> ON Semiconductor; manufacturer ON Semiconductor -> (none)
- R46, R47: Manufacturer (none) -> Stackpole Electronics; Part Number (none) -> RMCF0603JJ1K00
- U12: Manufacturer (none) -> Texas Instruments; manufacturer Texas Instruments -> (none)
Changed lines of the file:
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@@
       (effects (font (size 1.27 1.27)) (justify left) hide)
     )
-    (property "manufacturer" "ON Semiconductor" (id 18) (at 325.12 105.41 0)
+    (property "manufacturer" "" (id 18) (at 325.12 105.41 0)
       (effects (font (size 1.27 1.27)) (justify left) hide)
     )
@@
     )
     (property "Stock" "25" (id 35) (at 264.16 105.41 0)
+      (effects (font (size 1.27 1.27)) hide)
+    )
+    (property "Manufacturer" "ON Semiconductor" (id 36) (at 264.16 105.41 0)
       (effects (font (size 1.27 1.27)) hide)
     )
@@
       (effects (font (size 1.27 1.27)) (justify left) hide)
     )
-    (property "manufacturer" "Texas Instruments" (id 20) (at 158.75 71.12 0)
+    (property "manufacturer" "" (id 20) (at 158.75 71.12 0)
       (effects (font (size 1.27 1.27)) (justify left) hide)
     )
@@
     )
     (property "Stock" "25" (id 36) (at 158.75 127 0)
+      (effects (font (size 1.27 1.27)) hide)
+    )
+    (property "Manufacturer" "Texas Instruments" (id 37) (at 158.75 127 0)
       (effects (font (size 1.27 1.27)) hide)
     )
@@
       (effects (font (size 1.27 1.27)) hide)
     )
+    (property "Manufacturer" "Semitec" (id 6) (at 106.68 163.83 0)
+      (effects (font (size 1.27 1.27)) hide)
+    )
     (pin "1")
     (pin "2")
@@
       (effects (font (size 1.27 1.27)) hide)
     )
+    (property "Manufacturer" "Semitec" (id 6) (at 96.52 165.1 0)
+      (effects (font (size 1.27 1.27)) hide)
+    )
     (pin "1")
     (pin "2")
@@
       (effects (font (size 1.27 1.27)) hide)
     )
+    (property "Manufacturer" "Stackpole Electronics" (id 4) (at 264.16 114.3 0)
+      (effects (font (size 1.27 1.27)) hide)
+    )
+    (property "Part Number" "RMCF0603JJ1K00" (id 5) (at 264.16 114.3 0)
+      (effects (font (size 1.27 1.27)) hide)
+    )
     (pin "1")
     (pin "2")
@@
       (effects (font (size 1.27 1.27)) hide)
     )
+    (property "Manufacturer" "Stackpole Electronics" (id 4) (at 256.54 114.3 0)
+      (effects (font (size 1.27 1.27)) hide)
+    )
+    (property "Part Number" "RMCF0603JJ1K00" (id 5) (at 256.54 114.3 0)
+      (effects (font (size 1.27 1.27)) hide)
+    )

Commit message: Mainly just small value resistor tweaks and notes on their required power ratings.
Parts:
- R44: footprint Resistor_SMD:R_0603_1608Metric -> Resistor_SMD:R_0805_2012Metric
Changed lines of the file:
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@@
     (property "Reference" "R44" (id 0) (at 229.87 77.47 90))
     (property "Value" "5m" (id 1) (at 229.87 80.01 90))
-    (property "Footprint" "Resistor_SMD:R_0603_1608Metric" (id 2) (at 229.87 80.772 90)
+    (property "Footprint" "Resistor_SMD:R_0805_2012Metric" (id 2) (at 229.87 80.772 90)
       (effects (font (size 1.27 1.27)) hide)
     )
@@
       (effects (font (size 1.27 1.27)) hide)
     )
+    (property "Description" "Max Current 167 uA.  1/16W ok" (id 4) (at 120.65 110.49 0)
+      (effects (font (size 1.27 1.27)) hide)
+    )
     (pin "1")
     (pin "2")
@@
       (effects (font (size 1.27 1.27)) hide)
     )
+    (property "Description" "1/16W ok" (id 4) (at 120.65 124.46 0)
+      (effects (font (size 1.27 1.27)) hide)
+    )

Commit message: bulk BOM edits. Mainly dealing with cap voltage ratings and part selection
Parts:
- C55: Manufacturer (none) -> Samsung; Part Number (none) -> CL10A105KQ8NNNC
- C56: Manufacturer (none) -> Samsung; Part Number (none) -> CL10B474KO8NNNC
- C57, C58, C59, C60, C61, C62, C63, C64, C65, C66: Manufacturer (none) -> Samsung; Part Number (none) -> CL10B104KB8NNWC
- R41, R42: Manufacturer (none) -> Stackpole Electronics; Part Number (none) -> RMCF0603JT10R0
- R44: Manufacturer (none) -> Yageo; Part Number (none) -> PA0805FRF470R005L
Changed lines of the file:
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@@
+      (effects (font (size 1.27 1.27)) hide)
+    )
+    (property "Manufacturer" "Samsung" (id 4) (at 287.02 140.97 0)
+      (effects (font (size 1.27 1.27)) hide)
+    )
+    (property "Part Number" "CL10B104KB8NNWC" (id 5) (at 287.02 140.97 0)
       (effects (font (size 1.27 1.27)) hide)
     )
@@
     )
     (property "Datasheet" "~" (id 3) (at 267.97 71.12 0)
+      (effects (font (size 1.27 1.27)) hide)
+    )
+    (property "Manufacturer" "Samsung" (id 4) (at 267.97 71.12 0)
+      (effects (font (size 1.27 1.27)) hide)
+    )
+    (property "Part Number" "CL10B104KB8NNWC" (id 5) (at 267.97 71.12 0)
       (effects (font (size 1.27 1.27)) hide)
     )
@@
       (effects (font (size 1.27 1.27)) hide)
     )
+    (property "Manufacturer" "Samsung" (id 4) (at 312.42 133.35 0)
+      (effects (font (size 1.27 1.27)) hide)
+    )
+    (property "Part Number" "CL10B104KB8NNWC" (id 5) (at 312.42 133.35 0)
+      (effects (font (size 1.27 1.27)) hide)
+    )
     (pin "1")
     (pin "2")
@@
       (effects (font (size 1.27 1.27)) hide)
     )
+    (property "Manufacturer" "Samsung" (id 4) (at 222.25 106.68 0)
+      (effects (font (size 1.27 1.27)) hide)
+    )
+    (property "Part Number" "CL10B104KB8NNWC" (id 5) (at 222.25 106.68 0)
+      (effects (font (size 1.27 1.27)) hide)
+    )
     (pin "1")
     (pin "2")
@@
     )
     (property "Datasheet" "~" (id 3) (at 124.46 143.51 0)
+      (effects (font (size 1.27 1.27)) hide)
+    )
+    (property "Manufacturer" "Samsung" (id 4) (at 124.46 143.51 0)
+      (effects (font (size 1.27 1.27)) hide)
+    )
+    (property "Part Number" "CL10A105KQ8NNNC" (id 5) (at 124.46 143.51 0)
       (effects (font (size 1.27 1.27)) hide)
     )
@@
     )
     (property "Datasheet" "~" (id 3) (at 229.87 82.55 0)
+      (effects (font (size 1.27 1.27)) hide)
+    )
+    (property "Description" "1/2W" (id 4) (at 229.87 82.55 0)
+      (effects (font (size 1.27 1.27)) hide)
+    )
+    (property "Manufacturer" "Yageo" (id 5) (at 229.87 82.55 0)
+      (effects (font (size 1.27 1.27)) hide)
+    )
+    (property "Part Number" "PA0805FRF470R005L" (id 6) (at 229.87 82.55 0)
       (effects (font (size 1.27 1.27)) hide)
     )
@@
       (effects (font (size 1.27 1.27)) hide)
     )
+    (property "Manufacturer" "Samsung" (id 4) (at 234.95 106.68 0)
+      (effects (font (size 1.27 1.27)) hide)
+    )
+    (property "Part Number" "CL10B104KB8NNWC" (id 5) (at 234.95 106.68 0)
+      (effects (font (size 1.27 1.27)) hide)
+    )
     (pin "1")
     (pin "2")
@@
       (effects (font (size 1.27 1.27)) hide)
     )
+    (property "Manufacturer" "Samsung" (id 4) (at 252.73 71.12 0)
+      (effects (font (size 1.27 1.27)) hide)
+    )
+    (property "Part Number" "CL10B104KB8NNWC" (id 5) (at 252.73 71.12 0)
+      (effects (font (size 1.27 1.27)) hide)
+    )
     (pin "1")
     (pin "2")
@@
       (effects (font (size 1.27 1.27)) hide)
     )
+    (property "Manufacturer" "Samsung" (id 4) (at 147.32 114.3 0)
+      (effects (font (size 1.27 1.27)) hide)
+    )
+    (property "Part Number" "CL10B104KB8NNWC" (id 5) (at 147.32 114.3 0)
+      (effects (font (size 1.27 1.27)) hide)
+    )
     (pin "1")
     (pin "2")
@@
       (effects (font (size 1.27 1.27)) hide)
     )
+    (property "Manufacturer" "Samsung" (id 4) (at 312.42 146.05 0)
+      (effects (font (size 1.27 1.27)) hide)
+    )
+    (property "Part Number" "CL10B104KB8NNWC" (id 5) (at 312.42 146.05 0)
+      (effects (font (size 1.27 1.27)) hide)
+    )
     (pin "1")
     (pin "2")
@@
     )
     (property "Datasheet" "~" (id 3) (at 132.08 128.27 0)
+      (effects (font (size 1.27 1.27)) hide)
+    )
+    (property "Manufacturer" "Samsung" (id 4) (at 132.08 128.27 0)
+      (effects (font (size 1.27 1.27)) hide)
+    )
+    (property "Part Number" "CL10B104KB8NNWC" (id 5) (at 132.08 128.27 0)
       (effects (font (size 1.27 1.27)) hide)
     )
@@
       (effects (font (size 1.27 1.27)) hide)
     )
+    (property "Manufacturer" "Stackpole Electronics" (id 5) (at 120.65 110.49 0)
+      (effects (font (size 1.27 1.27)) hide)
+    )
+    (property "Part Number" "RMCF0603JT10R0" (id 6) (at 120.65 110.49 0)
+      (effects (font (size 1.27 1.27)) hide)
+    )
     (pin "1")
     (pin "2")
@@
       (effects (font (size 1.27 1.27)) hide)
     )
+    (property "Manufacturer" "Samsung" (id 4) (at 228.6 119.38 0)
+      (effects (font (size 1.27 1.27)) hide)
+    )
+    (property "Part Number" "CL10B104KB8NNWC" (id 5) (at 228.6 119.38 0)
+      (effects (font (size 1.27 1.27)) hide)
+    )
     (pin "1")
     (pin "2")
@@
       (effects (font (size 1.27 1.27)) hide)
     )
+    (property "Manufacturer" "Samsung" (id 4) (at 137.16 143.51 0)
+      (effects (font (size 1.27 1.27)) hide)
+    )
+    (property "Part Number" "CL10B474KO8NNNC" (id 5) (at 137.16 143.51 0)
+      (effects (font (size 1.27 1.27)) hide)
+    )
     (pin "1")
     (pin "2")
@@
       (effects (font (size 1.27 1.27)) hide)
     )
+    (property "Manufacturer" "Stackpole Electronics" (id 5) (at 120.65 124.46 0)
+      (effects (font (size 1.27 1.27)) hide)
+    )
+    (property "Part Number" "RMCF0603JT10R0" (id 6) (at 120.65 124.46 0)
+      (effects (font (size 1.27 1.27)) hide)
+    )
