File: kicad/robot/USB-PD-ExtChg.kicad_sch (KiCad schematic)
At the start: 32 parts, among them J1 USBC_Receptacle_SMD_RA, Q3 YJL3416A, Q4 YJL3416A, U18 AP33771DKZ-13, U25 TVS0500DRV, U26 TPD1E05U06, U27 TPD1E05U06, U28 TPD1E05U06, U29 TPD1E05U06

Commit message: updated all footprint fields in schematic symbols with local robot ones
Parts:
- C102, C103, C104, C105, C18, C19: footprint Capacitor_SMD:C_0402_1005Metric -> robot:C_0402_1005Metric
- C20: footprint Capacitor_SMD:C_0603_1608Metric -> robot:C_0603_1608Metric
- D4: footprint Diode_SMD:D_0603_1608Metric -> robot:D_0603_1608Metric
- J1: footprint AltiumImports:CON_USB3.1-C_RCPT_SMD_RA_ACP_12401610E4#2A -> robot:CON_USB3.1-C_RCPT_SMD_RA_ACP_12401610E4#2A
- Q3, Q4: footprint Package_TO_SOT_SMD:SOT-23 -> robot:SOT-23
- R51: footprint Resistor_SMD:R_1206_3216Metric -> robot:R_1206_3216Metric
- R57, R58, R59, R60, R61, R62, R63, R64, R66: footprint Resistor_SMD:R_0603_1608Metric -> robot:R_0603_1608Metric
- TP10, TP11, TP21, TP22, TP9: footprint TestPoint:KEYSTONE_5002 -> robot:KEYSTONE_5002
- U18: footprint Package_DFN_QFN:AP33771DKZ13 -> robot:AP33771DKZ13
- U25: footprint Package_SON:TVS0500DRVR -> robot:TVS0500DRVR
- U26, U27, U28, U29: footprint Package_X1SON:TPD1E05U06DPYR -> robot:TPD1E05U06DPYR
Changed lines of the file:
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@@
       (effects (font (size 1.27 1.27)) (justify left))
     )
-    (property "Footprint" "Capacitor_SMD:C_0603_1608Metric" (at 229.5652 137.16 0)
+    (property "Footprint" "robot:C_0603_1608Metric" (at 229.5652 137.16 0)
       (effects (font (size 1.27 1.27)) hide)
     )
@@
       (effects (font (size 1.27 1.27)) (justify right))
     )
-    (property "Footprint" "Resistor_SMD:R_0603_1608Metric" (at 283.972 213.36 90)
+    (property "Footprint" "robot:R_0603_1608Metric" (at 283.972 213.36 90)
       (effects (font (size 1.27 1.27)) hide)
     )
@@
       (effects (font (size 1.27 1.27)))
     )
-    (property "Footprint" "Package_DFN_QFN:AP33771DKZ13" (at 292.735 139.065 0)
+    (property "Footprint" "robot:AP33771DKZ13" (at 292.735 139.065 0)
       (effects (font (size 1.27 1.27)) (justify left) hide)
     )
@@
       (effects (font (size 1.27 1.27)))
     )
-    (property "Footprint" "Resistor_SMD:R_1206_3216Metric" (at 266.7 127.508 90)
+    (property "Footprint" "robot:R_1206_3216Metric" (at 266.7 127.508 90)
       (effects (font (size 1.27 1.27)) hide)
     )
@@
       (effects (font (size 1.27 1.27)) (justify left) hide)
     )
-    (property "Footprint" "TestPoint:KEYSTONE_5002" (at 212.09 184.15 0)
+    (property "Footprint" "robot:KEYSTONE_5002" (at 212.09 184.15 0)
       (effects (font (size 1.27 1.27)) hide)
     )
@@
       (effects (font (size 1.524 1.524)) hide)
     )
-    (property "Footprint" "Package_X1SON:TPD1E05U06DPYR" (at 236.22 264.16 0)
+    (property "Footprint" "robot:TPD1E05U06DPYR" (at 236.22 264.16 0)
       (effects (font (size 1.524 1.524)) hide)
     )
@@
       (effects (font (size 1.524 1.524)) hide)
     )
-    (property "Footprint" "Package_X1SON:TPD1E05U06DPYR" (at 203.2 264.16 0)
+    (property "Footprint" "robot:TPD1E05U06DPYR" (at 203.2 264.16 0)
       (effects (font (size 1.524 1.524)) hide)
     )
@@
       (effects (font (size 1.27 1.27)) (justify right))
     )
-    (property "Footprint" "Resistor_SMD:R_0603_1608Metric" (at 289.052 226.06 90)
+    (property "Footprint" "robot:R_0603_1608Metric" (at 289.052 226.06 90)
       (effects (font (size 1.27 1.27)) hide)
     )
@@
       (effects (font (size 1.524 1.524)) hide)
     )
-    (property "Footprint" "Package_X1SON:TPD1E05U06DPYR" (at 231.14 218.44 0)
+    (property "Footprint" "robot:TPD1E05U06DPYR" (at 231.14 218.44 0)
       (effects (font (size 1.524 1.524)) hide)
     )
@@
       (effects (font (size 1.27 1.27)) (justify left))
     )
-    (property "Footprint" "Resistor_SMD:R_0603_1608Metric" (at 311.912 199.39 90)
+    (property "Footprint" "robot:R_0603_1608Metric" (at 311.912 199.39 90)
       (effects (font (size 1.27 1.27)) hide)
     )
@@
       (effects (font (size 1.27 1.27)))
     )
-    (property "Footprint" "Package_TO_SOT_SMD:SOT-23" (at 297.815 123.19 0)
+    (property "Footprint" "robot:SOT-23" (at 297.815 123.19 0)
       (effects (font (size 1.27 1.27)) (justify left) hide)
     )
@@
       (effects (font (size 1.27 1.27)) (justify left))
     )
-    (property "Footprint" "Capacitor_SMD:C_0402_1005Metric" (at 299.4152 217.17 0)
+    (property "Footprint" "robot:C_0402_1005Metric" (at 299.4152 217.17 0)
       (effects (font (size 1.27 1.27)) hide)
     )
@@
       (effects (font (size 1.27 1.27)) (justify left))
     )
-    (property "Footprint" "Capacitor_SMD:C_0402_1005Metric" (at 190.1952 200.66 0)
+    (property "Footprint" "robot:C_0402_1005Metric" (at 190.1952 200.66 0)
       (effects (font (size 1.27 1.27)) hide)
     )
@@
       (effects (font (size 1.27 1.27)) (justify right))
     )
-    (property "Footprint" "Diode_SMD:D_0603_1608Metric" (at 263.525 207.01 0)
+    (property "Footprint" "robot:D_0603_1608Metric" (at 263.525 207.01 0)
       (effects (font (size 1.27 1.27)) hide)
     )
@@
       (effects (font (size 1.27 1.27)) (justify left))
     )
-    (property "Footprint" "Capacitor_SMD:C_0402_1005Metric" (at 202.8952 200.66 0)
+    (property "Footprint" "robot:C_0402_1005Metric" (at 202.8952 200.66 0)
       (effects (font (size 1.27 1.27)) hide)
     )
@@
       (effects (font (size 1.27 1.27)) (justify left))
     )
-    (property "Footprint" "Resistor_SMD:R_0603_1608Metric" (at 287.782 152.4 90)
+    (property "Footprint" "robot:R_0603_1608Metric" (at 287.782 152.4 90)
       (effects (font (size 1.27 1.27)) hide)
     )
@@
       (effects (font (size 1.524 1.524)) hide)
     )
-    (property "Footprint" "Package_X1SON:TPD1E05U06DPYR" (at 250.19 218.44 0)
+    (property "Footprint" "robot:TPD1E05U06DPYR" (at 250.19 218.44 0)
       (effects (font (size 1.524 1.524)) hide)
     )
@@
       (effects (font (size 1.27 1.27)) (justify left bottom) hide)
     )
-    (property "Footprint" "AltiumImports:CON_USB3.1-C_RCPT_SMD_RA_ACP_12401610E4#2A" (at 177.8 116.84 0)
+    (property "Footprint" "robot:CON_USB3.1-C_RCPT_SMD_RA_ACP_12401610E4#2A" (at 177.8 116.84 0)
       (effects (font (size 1.27 1.27)) hide)
     )
@@
       (effects (font (size 1.27 1.27)) (justify left) hide)
     )
-    (property "Footprint" "TestPoint:KEYSTONE_5002" (at 241.3 125.73 0)
+    (property "Footprint" "robot:KEYSTONE_5002" (at 241.3 125.73 0)
       (effects (font (size 1.27 1.27)) hide)
     )
@@
       (effects (font (size 1.27 1.27)) (justify left) hide)
     )
-    (property "Footprint" "TestPoint:KEYSTONE_5002" (at 228.6 247.65 0)
+    (property "Footprint" "robot:KEYSTONE_5002" (at 228.6 247.65 0)
       (effects (font (size 1.27 1.27)) hide)
     )
@@
       (effects (font (size 1.27 1.27)) (justify left))
     )
-    (property "Footprint" "Capacitor_SMD:C_0402_1005Metric" (at 337.5152 135.255 0)
+    (property "Footprint" "robot:C_0402_1005Metric" (at 337.5152 135.255 0)
       (effects (font (size 1.27 1.27)) hide)
     )
@@
       (effects (font (size 1.27 1.27)) (justify left))
     )
-    (property "Footprint" "Resistor_SMD:R_0603_1608Metric" (at 335.407 193.04 90)
+    (property "Footprint" "robot:R_0603_1608Metric" (at 335.407 193.04 90)
       (effects (font (size 1.27 1.27)) hide)
     )
@@
       (effects (font (size 1.27 1.27)) (justify right))
     )
-    (property "Footprint" "Resistor_SMD:R_0603_1608Metric" (at 294.132 237.49 90)
+    (property "Footprint" "robot:R_0603_1608Metric" (at 294.132 237.49 90)
       (effects (font (size 1.27 1.27)) hide)
     )
@@
       (effects (font (size 1.27 1.27)) (justify left) hide)
     )
-    (property "Footprint" "TestPoint:KEYSTONE_5002" (at 195.58 247.65 0)
+    (property "Footprint" "robot:KEYSTONE_5002" (at 195.58 247.65 0)
       (effects (font (size 1.27 1.27)) hide)
     )
@@
       (effects (font (size 1.27 1.27)) (justify left))
     )
-    (property "Footprint" "Capacitor_SMD:C_0402_1005Metric" (at 317.8302 173.355 0)
+    (property "Footprint" "robot:C_0402_1005Metric" (at 317.8302 173.355 0)
       (effects (font (size 1.27 1.27)) hide)
     )
@@
       (effects (font (size 1.27 1.27)) (justify left))
     )
-    (property "Footprint" "Resistor_SMD:R_0603_1608Metric" (at 261.747 198.12 90)
+    (property "Footprint" "robot:R_0603_1608Metric" (at 261.747 198.12 90)
       (effects (font (size 1.27 1.27)) hide)
     )
@@
       (effects (font (size 1.27 1.27)) (justify left) hide)
     )
-    (property "Footprint" "Package_SON:TVS0500DRVR" (at 234.315 133.985 0)
+    (property "Footprint" "robot:TVS0500DRVR" (at 234.315 133.985 0)
       (effects (font (size 1.27 1.27)) hide)
     )
@@
       (effects (font (size 1.27 1.27)))
     )
-    (property "Footprint" "Package_TO_SOT_SMD:SOT-23" (at 316.865 123.19 0)
+    (property "Footprint" "robot:SOT-23" (at 316.865 123.19 0)
       (effects (font (size 1.27 1.27)) (justify left) hide)
     )
@@
       (effects (font (size 1.27 1.27)) (justify left))
     )
-    (property "Footprint" "Capacitor_SMD:C_0402_1005Metric" (at 324.1802 198.755 0)
+    (property "Footprint" "robot:C_0402_1005Metric" (at 324.1802 198.755 0)
       (effects (font (size 1.27 1.27)) hide)
     )
@@
       (effects (font (size 1.27 1.27)) (justify left))
     )
-    (property "Footprint" "Resistor_SMD:R_0603_1608Metric" (at 305.562 129.54 90)
+    (property "Footprint" "robot:R_0603_1608Metric" (at 305.562 129.54 90)
       (effects (font (size 1.27 1.27)) hide)
     )
@@
       (effects (font (size 1.27 1.27)) (justify right) hide)
     )
-    (property "Footprint" "TestPoint:KEYSTONE_5002" (at 201.93 186.69 0)
+    (property "Footprint" "robot:KEYSTONE_5002" (at 201.93 186.69 0)
       (effects (font (size 1.27 1.27)) hide)
     )
@@
       (effects (font (size 1.27 1.27)) (justify left))
     )
-    (property "Footprint" "Resistor_SMD:R_0603_1608Metric" (at 344.297 193.04 90)
-      (effects (font (size 1.27 1.27)) hide)
-    )
+    (property "Footprint" "robot:R_0603_1608Metric" (at 344.297 193.04 90)
+      (effects (font (size 1.27 1.27)) hide)
+    )

Commit message: Exported all schematic symbols to local robot and refer to them in all symbols
Parts:
- C102, C103, C104, C105, C18, C19, C20: symbol Device:C -> robot:C
- D4: symbol Device:LED -> robot:LED
- J1: symbol Connector:0_mirrored_USBC_Receptacle_SMD_RA -> robot:0_mirrored_USBC_Receptacle_SMD_RA
- Q3, Q4: symbol Transistor_FET:YJL3416A -> robot:YJL3416A
- R51, R57, R58, R59, R60, R61, R62, R63, R64, R66: symbol Device:R -> robot:R
- TP10, TP11, TP21, TP22, TP9: symbol Connector:TestPoint -> robot:TestPoint
- U18: symbol Battery_Management:AP33771DKZ-13 -> robot:AP33771DKZ-13
- U25: symbol Power_Protection:TVS0500DRV -> robot:TVS0500DRV
- U26, U27, U28: symbol Diode:TPD1E05U06 -> robot:TPD1E05U06
- U29: symbol Diode:TPD1E05U06 -> robot:TPD1E05U06_1
Changed lines of the file:
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@@
     (effects (font (size 1.27 1.27)) (justify right))
   )
-  (symbol (lib_id "Device:C") (at 228.6 133.35 0) (unit 1)
+  (symbol (lib_id "robot:C") (at 228.6 133.35 0) (unit 1)
     (in_bom yes) (on_board yes) (dnp no)
     (property "Reference" "C20" (at 232.41 132.0799 0)
@@
     )
   )
-  (symbol (lib_id "Device:R") (at 285.75 213.36 0) (mirror x) (unit 1)
+  (symbol (lib_id "robot:R") (at 285.75 213.36 0) (mirror x) (unit 1)
     (in_bom yes) (on_board yes) (dnp no) (fields_autoplaced)
     (property "Reference" "R59" (at 283.21 212.0899 0)
@@
     )
   )
-  (symbol (lib_id "Battery_Management:AP33771DKZ-13") (at 292.1 187.96 0) (unit 1)
+  (symbol (lib_id "robot:AP33771DKZ-13") (at 292.1 187.96 0) (unit 1)
     (in_bom yes) (on_board yes) (dnp no)
     (property "Reference" "U18" (at 290.83 186.69 0)
@@
     )
   )
-  (symbol (lib_id "Device:R") (at 266.7 125.73 90) (unit 1)
+  (symbol (lib_id "robot:R") (at 266.7 125.73 90) (unit 1)
     (in_bom yes) (on_board yes) (dnp no) (fields_autoplaced)
     (property "Reference" "R51" (at 266.7 119.38 90)
@@
     )
   )
-  (symbol (lib_id "Connector:TestPoint") (at 207.01 184.15 0) (unit 1)
+  (symbol (lib_id "robot:TestPoint") (at 207.01 184.15 0) (unit 1)
     (in_bom yes) (on_board yes) (dnp no)
     (property "Reference" "TP9" (at 209.55 179.07 0)
@@
     )
   )
-  (symbol (lib_name "TPD1E05U06_1") (lib_id "Diode:TPD1E05U06") (at 236.22 247.65 0) (unit 1)
+  (symbol (lib_name "TPD1E05U06_1") (lib_id "robot:TPD1E05U06_1") (at 236.22 247.65 0) (unit 1)
     (in_bom yes) (on_board yes) (dnp no)
     (property "Reference" "U29" (at 229.87 236.22 0)
@@
     )
   )
-  (symbol (lib_id "Diode:TPD1E05U06") (at 203.2 247.65 0) (unit 1)
+  (symbol (lib_id "robot:TPD1E05U06") (at 203.2 247.65 0) (unit 1)
     (in_bom yes) (on_board yes) (dnp no)
     (property "Reference" "U28" (at 196.85 236.22 0)
@@
     )
   )
-  (symbol (lib_id "Device:R") (at 290.83 226.06 0) (mirror x) (unit 1)
+  (symbol (lib_id "robot:R") (at 290.83 226.06 0) (mirror x) (unit 1)
     (in_bom yes) (on_board yes) (dnp no) (fields_autoplaced)
     (property "Reference" "R60" (at 288.29 224.7899 0)
@@
     )
   )
-  (symbol (lib_id "Diode:TPD1E05U06") (at 231.14 201.93 0) (unit 1)
+  (symbol (lib_id "robot:TPD1E05U06") (at 231.14 201.93 0) (unit 1)
     (in_bom yes) (on_board yes) (dnp no)
     (property "Reference" "U26" (at 224.79 190.5 0)
@@
     )
   )
-  (symbol (lib_id "Device:R") (at 313.69 199.39 0) (unit 1)
+  (symbol (lib_id "robot:R") (at 313.69 199.39 0) (unit 1)
     (in_bom yes) (on_board yes) (dnp no) (fields_autoplaced)
     (property "Reference" "R62" (at 315.468 198.5553 0)
@@
     )
   )
-  (symbol (lib_id "Transistor_FET:YJL3416A") (at 295.91 128.27 90) (unit 1)
+  (symbol (lib_id "robot:YJL3416A") (at 295.91 128.27 90) (unit 1)
     (in_bom yes) (on_board yes) (dnp no) (fields_autoplaced)
     (property "Reference" "Q3" (at 296.6085 118.11 90)
@@
     )
   )
-  (symbol (lib_id "Device:C") (at 298.45 213.36 0) (unit 1)
+  (symbol (lib_id "robot:C") (at 298.45 213.36 0) (unit 1)
     (in_bom yes) (on_board yes) (dnp no)
     (property "Reference" "C102" (at 302.26 212.0899 0)
@@
     )
   )
-  (symbol (lib_id "Device:C") (at 189.23 196.85 0) (unit 1)
+  (symbol (lib_id "robot:C") (at 189.23 196.85 0) (unit 1)
     (in_bom yes) (on_board yes) (dnp no)
     (property "Reference" "C18" (at 192.532 195.58 0)
@@
     )
   )
-  (symbol (lib_id "Device:LED") (at 263.525 207.01 90) (unit 1)
+  (symbol (lib_id "robot:LED") (at 263.525 207.01 90) (unit 1)
     (in_bom yes) (on_board yes) (dnp no) (fields_autoplaced)
     (property "Reference" "D4" (at 267.335 207.3274 90)
@@
     )
   )
-  (symbol (lib_id "Device:C") (at 201.93 196.85 0) (unit 1)
+  (symbol (lib_id "robot:C") (at 201.93 196.85 0) (unit 1)
     (in_bom yes) (on_board yes) (dnp no)
     (property "Reference" "C19" (at 205.74 195.5799 0)
@@
     )
   )
-  (symbol (lib_id "Device:R") (at 289.56 152.4 0) (unit 1)
+  (symbol (lib_id "robot:R") (at 289.56 152.4 0) (unit 1)
     (in_bom yes) (on_board yes) (dnp no) (fields_autoplaced)
     (property "Reference" "R58" (at 292.1 151.1299 0)
@@
     )
   )
-  (symbol (lib_id "Diode:TPD1E05U06") (at 250.19 201.93 0) (unit 1)
+  (symbol (lib_id "robot:TPD1E05U06") (at 250.19 201.93 0) (unit 1)
     (in_bom yes) (on_board yes) (dnp no)
     (property "Reference" "U27" (at 243.84 190.5 0)
@@
     )
   )
-  (symbol (lib_id "Connector:0_mirrored_USBC_Receptacle_SMD_RA") (at 177.8 116.84 0) (unit 1)
+  (symbol (lib_id "robot:0_mirrored_USBC_Receptacle_SMD_RA") (at 177.8 116.84 0) (unit 1)
     (in_bom yes) (on_board yes) (dnp no)
     (property "Reference" "J1" (at 160.02 116.84 0)
@@
     )
   )
-  (symbol (lib_id "Connector:TestPoint") (at 236.22 125.73 0) (unit 1)
+  (symbol (lib_id "robot:TestPoint") (at 236.22 125.73 0) (unit 1)
     (in_bom yes) (on_board yes) (dnp no)
     (property "Reference" "TP11" (at 238.76 120.65 0)
@@
     )
   )
-  (symbol (lib_id "Connector:TestPoint") (at 223.52 247.65 0) (unit 1)
+  (symbol (lib_id "robot:TestPoint") (at 223.52 247.65 0) (unit 1)
     (in_bom yes) (on_board yes) (dnp no)
     (property "Reference" "TP22" (at 226.06 242.57 0)
@@
     )
   )
-  (symbol (lib_id "Device:C") (at 336.55 131.445 0) (unit 1)
+  (symbol (lib_id "robot:C") (at 336.55 131.445 0) (unit 1)
     (in_bom yes) (on_board yes) (dnp no)
     (property "Reference" "C105" (at 340.36 130.1749 0)
@@
     )
   )
-  (symbol (lib_id "Device:R") (at 337.185 193.04 0) (unit 1)
+  (symbol (lib_id "robot:R") (at 337.185 193.04 0) (unit 1)
     (in_bom yes) (on_board yes) (dnp no) (fields_autoplaced)
     (property "Reference" "R63" (at 339.725 191.7699 0)
@@
     )
   )
-  (symbol (lib_id "Device:R") (at 295.91 237.49 0) (mirror x) (unit 1)
+  (symbol (lib_id "robot:R") (at 295.91 237.49 0) (mirror x) (unit 1)
     (in_bom yes) (on_board yes) (dnp no) (fields_autoplaced)
     (property "Reference" "R61" (at 293.37 236.2199 0)
@@
     )
   )
-  (symbol (lib_id "Connector:TestPoint") (at 190.5 247.65 0) (unit 1)
+  (symbol (lib_id "robot:TestPoint") (at 190.5 247.65 0) (unit 1)
     (in_bom yes) (on_board yes) (dnp no) (fields_autoplaced)
     (property "Reference" "TP21" (at 193.04 243.0779 0)
@@
     )
   )
-  (symbol (lib_id "Device:C") (at 316.865 169.545 0) (unit 1)
+  (symbol (lib_id "robot:C") (at 316.865 169.545 0) (unit 1)
     (in_bom yes) (on_board yes) (dnp no)
     (property "Reference" "C103" (at 320.675 168.2749 0)
@@
     )
   )
-  (symbol (lib_id "Device:R") (at 263.525 198.12 0) (unit 1)
+  (symbol (lib_id "robot:R") (at 263.525 198.12 0) (unit 1)
     (in_bom yes) (on_board yes) (dnp no) (fields_autoplaced)
     (property "Reference" "R57" (at 265.303 197.2853 0)
@@
     )
   )
-  (symbol (lib_id "Power_Protection:TVS0500DRV") (at 210.82 134.62 0) (unit 1)
+  (symbol (lib_id "robot:TVS0500DRV") (at 210.82 134.62 0) (unit 1)
     (in_bom yes) (on_board yes) (dnp no) (fields_autoplaced)
     (property "Reference" "U25" (at 214.63 134.6199 0)
@@
     )
   )
-  (symbol (lib_id "Transistor_FET:YJL3416A") (at 318.77 128.27 270) (mirror x) (unit 1)
+  (symbol (lib_id "robot:YJL3416A") (at 318.77 128.27 270) (mirror x) (unit 1)
     (in_bom yes) (on_board yes) (dnp no) (fields_autoplaced)
     (property "Reference" "Q4" (at 318.0715 118.11 90)
@@
     )
   )
-  (symbol (lib_id "Device:C") (at 323.215 194.945 0) (unit 1)
+  (symbol (lib_id "robot:C") (at 323.215 194.945 0) (unit 1)
     (in_bom yes) (on_board yes) (dnp no)
     (property "Reference" "C104" (at 327.025 193.6749 0)
@@
     )
   )
-  (symbol (lib_id "Device:R") (at 307.34 129.54 0) (unit 1)
+  (symbol (lib_id "robot:R") (at 307.34 129.54 0) (unit 1)
     (in_bom no) (on_board yes) (dnp yes) (fields_autoplaced)
     (property "Reference" "R66" (at 309.88 128.2699 0)
@@
     )
   )
-  (symbol (lib_id "Connector:TestPoint") (at 207.01 186.69 180) (unit 1)
+  (symbol (lib_id "robot:TestPoint") (at 207.01 186.69 180) (unit 1)
     (in_bom yes) (on_board yes) (dnp no)
     (property "Reference" "TP10" (at 209.55 189.23 0)
@@
     )
   )
-  (symbol (lib_id "Device:R") (at 346.075 193.04 0) (unit 1)
+  (symbol (lib_id "robot:R") (at 346.075 193.04 0) (unit 1)
     (in_bom yes) (on_board yes) (dnp no) (fields_autoplaced)
     (property "Reference" "R64" (at 348.615 191.7699 0)
